File: eagle/projekt/schema.sch (EAGLE design)
At the start: 21 parts, among them IC1 ESP12E_DEVKIT, IC2 LF50CP, J1 PSH02-02W, Q2 BC847CSMD

Commit message: Schema
Parts:
- removed C5: 100n/100V, parts_mix:C-EU025-025X050
- removed C6: 100u/25V, parts_mix:CPOL-EUE5-13
- removed C7: 100u/25V, parts_mix:CPOL-EUE3.5-8
- removed U$1, U$2: (no value), level_shifter:LEVEL_SHIFTER
- added C1: 100n/100V, parts:C-EUC025-025X050
- added C2: 10u/25V, parts:CPOL-EUE3,5-8
- added C3: 100u/25V, parts:CPOL-EUE5-13
- added IC3, IC4: LEVEL_SHIFTER, level_shifter:LEVEL_SHIFTER
- added R7: 470, rcl:R-EU_R1206
- added S2: DTS-6, switch-tact:DTS-6
- C4: device rcl:C-EU025-025X050 -> parts:C-EUC025-025X050
- IC2: device parts_mix:LF50CP -> parts:LF50CP
- PL1: device parts_mix:14V -> parts:14V
Connections:
- new net 3.3V: IC1.3V3@0, IC1.3V3@1, IC1.3V3@2, IC3.LV, IC4.LV
- new net 5V: C2.+, C4.1, IC1.VIN, IC2.VO, IC3.HV, IC4.HV, R1.2, S1.4
- new net ADC: R5.1
- new net D0: IC1.D0, IC3.LV1
- new net D1: IC1.D1, IC3.LV2
- new net D2: IC1.D2, IC3.LV3
- new net D5: IC1.D5, IC3.LV4
- new net D6: IC1.D6, IC4.LV1
- new net D7: IC1.D7, IC4.LV2, S1.2
- new net GND: C1.2, C2.-, C3.-, C4.2, IC1.GND@0, IC1.GND@1, IC1.GND@2, IC1.GND@3, IC2.GND, IC3.GND@0, IC3.GND@1, IC4.GND@0, IC4.GND@1, J1-1.S, LED1.C, Q2.E, R4.1, R6.2, S2.1, S2.2
- new net GPIO1: IC4.HV4
- new net GPIO12: IC4.HV1
- new net GPIO13: IC4.HV2
- new net GPIO14: IC3.HV4
- new net GPIO16: IC3.HV1
- new net GPIO3: IC4.HV3
- new net GPIO4: IC3.HV3
- new net GPIO5: IC3.HV2
- new net N$1: IC1.AD0, R5.2, R6.1
- new net N$14: C1.1, C3.+, D1.C, IC2.VI, J1-2.S
- new net N$2: LED1.A, R2.2
- new net N$3: R2.1, S1.1
- new net N$4: R7.1, S2.3, S2.4
- new net N$5: R3.1, S1.3
- new net N$6: Q2.B, R3.2, R4.2
- new net N$8: LED2.C, Q2.C
- new net N$9: LED2.A, R1.1
- new net RST: IC1.RST, R7.2
- new net RX: IC1.RX, IC4.LV3
- new net TX: IC1.TX, IC4.LV4
- new net VIN: D1.A
Other:
- moved on the sheet: C4, LED1, LED2, PL1, Q2, R1, R2, R3, R4, R5, R6, S1

Commit message: Schema
Connections:
- new net N$10: PL1.13
- new net N$11: PL1.2
- new net N$7: PL1.1
- net ADC: now also PL1.12
- net GND: now also PL1.14
- net GPIO1: now also PL1.3
- net GPIO12: now also PL1.7
- net GPIO13: now also PL1.8
- net GPIO14: now also PL1.9
- net GPIO16: now also PL1.10
- net GPIO3: now also PL1.4
- net GPIO4: now also PL1.5
- net GPIO5: now also PL1.6
- net RST: now also PL1.11
Other:
- note added: "+3.3V"
- note added: "+5V"
- note added: "1"
- note added: "14"
- note added: "2"
- note added: "ADC"
- note added: "GND"
- note added: "GPIO1/TX"
- note added: "GPIO12"
- note added: "GPIO13"
- note added: "GPIO14"
- note added: "GPIO16"
- note added: "GPIO3/RX"
- note added: "GPIO4"
- note added: "GPIO5"
- note added: "RST"
- note added: "VIN"

Commit message: Schema
Connections:
- removed net N$10: PL1.13
- removed net N$11: PL1.2
- removed net N$7: PL1.1
- net 3.3V: now also PL1.2
- net 5V: now also PL1.1
- net VIN: now also PL1.13
Changed lines of the file:
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@@
 <part name="GND8" library="supply1" deviceset="GND" device=""/>
 <part name="GND9" library="supply1" deviceset="GND" device=""/>
-<part name="GND10" library="supply1" deviceset="GND" device=""/>
 <part name="GND11" library="supply1" deviceset="GND" device=""/>
 <part name="GND12" library="supply1" deviceset="GND" device=""/>
@@
 <part name="IC4" library="level_shifter" deviceset="LEVEL_SHIFTER" device=""/>
 <part name="SUPPLY2" library="parts" deviceset="VIN" device=""/>
-<part name="SUPPLY3" library="parts" deviceset="VIN" device=""/>
-<part name="SUPPLY4" library="parts" deviceset="3.3V" device=""/>
 <part name="SUPPLY5" library="parts" deviceset="3.3V" device=""/>
 <part name="SUPPLY6" library="parts" deviceset="3.3V" device=""/>
@@
 <part name="SUPPLY10" library="parts" deviceset="5V" device=""/>
 <part name="SUPPLY11" library="parts" deviceset="5V" device=""/>
-<part name="SUPPLY12" library="parts" deviceset="5V" device=""/>
 <part name="SUPPLY14" library="parts" deviceset="5V" device=""/>
 <part name="GND4" library="supply1" deviceset="GND" device=""/>
@@
 <part name="GND14" library="supply1" deviceset="GND" device=""/>
 <part name="SUPPLY16" library="parts" deviceset="5V" device=""/>
+<part name="SUPPLY3" library="parts" deviceset="5V" device=""/>
+<part name="SUPPLY4" library="parts" deviceset="VIN" device=""/>
+<part name="SUPPLY12" library="parts" deviceset="3.3V" device=""/>
+<part name="GND10" library="supply1" deviceset="GND" device=""/>
 </parts>
 <sheets>
@@
 <instance part="GND8" gate="1" x="76.2" y="132.08"/>
 <instance part="GND9" gate="1" x="147.32" y="109.22"/>
-<instance part="GND10" gate="1" x="215.9" y="86.36"/>
 <instance part="GND11" gate="1" x="30.48" y="50.8"/>
 <instance part="GND12" gate="1" x="73.66" y="50.8"/>
@@
 <instance part="IC4" gate="G$1" x="124.46" y="55.88" rot="R180"/>
 <instance part="SUPPLY2" gate="G$1" x="38.1" y="165.1"/>
-<instance part="SUPPLY3" gate="G$1" x="195.58" y="122.555"/>
-<instance part="SUPPLY4" gate="G$1" x="218.44" y="122.555"/>
 <instance part="SUPPLY5" gate="G$1" x="76.2" y="101.6"/>
 <instance part="SUPPLY6" gate="G$1" x="27.94" y="83.82"/>
@@
 <instance part="SUPPLY10" gate="G$1" x="22.86" y="83.82"/>
 <instance part="SUPPLY11" gate="G$1" x="142.24" y="101.6"/>
-<instance part="SUPPLY12" gate="G$1" x="193.04" y="122.555"/>
 <instance part="SUPPLY14" gate="G$1" x="142.24" y="66.04"/>
 <instance part="GND4" gate="1" x="38.1" y="132.08"/>
@@
 <instance part="GND14" gate="1" x="167.64" y="132.08"/>
 <instance part="SUPPLY16" gate="G$1" x="147.32" y="165.1"/>
+<instance part="SUPPLY3" gate="G$1" x="193.04" y="119.38"/>
+<instance part="SUPPLY4" gate="G$1" x="195.58" y="119.38"/>
+<instance part="SUPPLY12" gate="G$1" x="215.9" y="119.38"/>
+<instance part="GND10" gate="1" x="215.9" y="86.36"/>
 </instances>
 <busses>
@@
 <segment>
 <pinref part="PL1" gate="G$1" pin="14"/>
+<pinref part="GND10" gate="1" pin="GND"/>
 <wire x1="213.36" y1="96.52" x2="215.9" y2="96.52" width="0.1524" layer="91"/>
-<pinref part="GND10" gate="1" pin="GND"/>
 <wire x1="215.9" y1="96.52" x2="215.9" y2="88.9" width="0.1524" layer="91"/>
 </segment>
@@
 </segment>
 <segment>
-<pinref part="SUPPLY3" gate="G$1" pin="VIN"/>
-<pinref part="SUPPLY3" gate="G$1" pin="VIN"/>
+<pinref part="PL1" gate="G$1" pin="13"/>
+<pinref part="SUPPLY4" gate="G$1" pin="VIN"/>
+<wire x1="198.12" y1="96.52" x2="195.58" y2="96.52" width="0.1524" layer="91"/>
+<wire x1="195.58" y1="96.52" x2="195.58" y2="119.38" width="0.1524" layer="91"/>
 </segment>
 </net>
@@
 <pinref part="SUPPLY16" gate="G$1" pin="5V"/>
 <wire x1="147.32" y1="160.02" x2="147.32" y2="165.1" width="0.1524" layer="91"/>
+</segment>
+<segment>
+<pinref part="PL1" gate="G$1" pin="1"/>
+<pinref part="SUPPLY3" gate="G$1" pin="5V"/>
+<wire x1="198.12" y1="111.76" x2="193.04" y2="111.76" width="0.1524" layer="91"/>
+<wire x1="193.04" y1="111.76" x2="193.04" y2="119.38" width="0.1524" layer="91"/>
 </segment>
 </net>
@@
 <wire x1="106.68" y1="55.88" x2="106.68" y2="66.04" width="0.1524" layer="91"/>
 </segment>
+<segment>
+<pinref part="PL1" gate="G$1" pin="2"/>
+<pinref part="SUPPLY12" gate="G$1" pin="3.3V"/>
+<wire x1="213.36" y1="111.76" x2="215.9" y2="111.76" width="0.1524" layer="91"/>
+<wire x1="215.9" y1="111.76" x2="215.9" y2="119.38" width="0.1524" layer="91"/>
+</segment>
 </net>
 <net name="N$5" class="0">
@@
 </segment>
 </net>
-<net name="N$7" class="0">
-<segment>
-<wire x1="193.04" y1="121.92" x2="193.04" y2="111.76" width="0.1524" layer="91"/>
-<pinref part="PL1" gate="G$1" pin="1"/>
-<wire x1="193.04" y1="111.76" x2="198.12" y2="111.76" width="0.1524" layer="91"/>
-</segment>
-</net>
-<net name="N$10" class="0">
-<segment>
-<wire x1="195.58" y1="121.92" x2="195.58" y2="96.52" width="0.1524" layer="91"/>
-<pinref part="PL1" gate="G$1" pin="13"/>
-<wire x1="195.58" y1="96.52" x2="198.12" y2="96.52" width="0.1524" layer="91"/>
-</segment>
-</net>
-<net name="N$11" class="0">
-<segment>
-<wire x1="218.44" y1="121.92" x2="218.44" y2="111.76" width="0.1524" layer="91"/>
-<pinref part="PL1" gate="G$1" pin="2"/>
-<wire x1="218.44" y1="111.76" x2="213.36" y2="111.76" width="0.1524" layer="91"/>
-</segment>
-</net>

Commit message: Schema
Parts:
- removed Q2: BC847CSMD, transistor-npn:BC847CSMD
- removed R6: 110k 1%, rcl:R-EU_R1206
- removed R7: 470, rcl:R-EU_R1206
- R1: value 1k6 -> 750
- R3: value 10k -> 56k 1%
- R4: value 200k -> 110k 1%
- R5: value 56k 1% -> 470
Connections:
- removed net N$6 (its old number): Q2.B, R3.2, R4.2
- removed net N$8: LED2.C, Q2.C
- new net D4: IC1.D4, LED2.C
- net 3.3V: now also S1.3
- net 5V: no longer R1.2
- net ADC: now also R3.1; no longer R5.1
- net D7: no longer S1.2
- net GND: now also R4.2; no longer Q2.E, R4.1, R6.2
- net N$1: now also R3.2, R4.1; no longer R5.2, R6.1
- net N$2: now also R2.1; no longer R2.2
- net N$3: now also R2.2; no longer R2.1
- net N$4: now also R5.1; no longer R7.1
- net N$5: now also R1.2, S1.2; no longer R3.1, S1.3
- net RST: now also R5.2; no longer R7.2
Other:
- moved on the sheet: LED2, R1, R2, R3, R4, R5, S1
