File: eagle/projekt/projekt.sch (EAGLE design)
At the start: 20 parts, among them IC1 ESP12E_DEVKIT, IC2 LF50CP, IC3 LEVEL_SHIFTER, IC4 LEVEL_SHIFTER, J1 PSH02-02W

Commit message: Board
Parts:
- PL1: device parts:14V -> parts:14H
Changed lines of the file:
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@@
 <part name="R4" library="rcl" deviceset="R-EU_" device="R1206" value="110k 1%"/>
 <part name="IC2" library="parts" deviceset="LF50" device="CP"/>
-<part name="PL1" library="parts" deviceset="14V" device=""/>
+<part name="PL1" library="parts" deviceset="14H" device=""/>
 <part name="C1" library="parts" deviceset="C-EU" device="C025-025X050" value="100n/100V"/>
 <part name="C2" library="parts" deviceset="CPOL-EU" device="E3,5-8" value="10u/25V"/>
