File: eagle/projekt/projekt.brd (EAGLE design)
At the start: 82 x 84 mm, 20 parts, among them IC1 ESP12E_DEVKIT, IC2 LF50CP, IC3 LEVEL_SHIFTER, IC4 LEVEL_SHIFTER, J1 PSH02-02W

Commit message: Board
Routing:
- net GND: track 375.8 -> 376.6 mm
- added copper zone on layer 16, net N$7
- added copper zone on layer 1, net N$8
Changed lines of the file:
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@@
 <board>
 <plain>
-<wire x1="0" y1="0" x2="82" y2="0" width="0" layer="20"/>
-<wire x1="82" y1="0" x2="82" y2="68" width="0" layer="20"/>
-<wire x1="0" y1="68" x2="0" y2="0" width="0" layer="20"/>
+<wire x1="0" y1="0" x2="82" y2="0" width="0.3048" layer="20"/>
+<wire x1="82" y1="0" x2="82" y2="68" width="0.3048" layer="20"/>
+<wire x1="0" y1="68" x2="0" y2="0" width="0.3048" layer="20"/>
 <hole x="4" y="10" drill="2.2"/>
 <hole x="78" y="10" drill="2.2"/>
 <hole x="78" y="64" drill="2.2"/>
 <hole x="4" y="64" drill="2.2"/>
-<wire x1="0" y1="68" x2="8" y2="68" width="0" layer="20"/>
-<wire x1="82" y1="68" x2="74" y2="68" width="0" layer="20"/>
-<wire x1="74" y1="68" x2="74" y2="84" width="0" layer="20"/>
-<wire x1="74" y1="84" x2="8" y2="84" width="0" layer="20"/>
-<wire x1="8" y1="84" x2="8" y2="68" width="0" layer="20"/>
+<wire x1="0" y1="68" x2="8" y2="68" width="0.3048" layer="20"/>
+<wire x1="82" y1="68" x2="74" y2="68" width="0.3048" layer="20"/>
+<wire x1="74" y1="68" x2="74" y2="84" width="0.3048" layer="20"/>
+<wire x1="74" y1="84" x2="8" y2="84" width="0.3048" layer="20"/>
+<wire x1="8" y1="84" x2="8" y2="68" width="0.3048" layer="20"/>
 <hole x="13.208" y="80.772" drill="2.8"/>
 <hole x="42.672" y="80.772" drill="2.8"/>
@@
 <wire x1="73.3298" y1="64.77" x2="73.3425" y2="64.77" width="0.6096" layer="16"/>
 <wire x1="73.3298" y1="64.77" x2="71.12" y2="64.77" width="0.8128" layer="16"/>
-<wire x1="71.12" y1="74.93" x2="73.025" y2="74.93" width="0.6096" layer="16"/>
-<wire x1="64.135" y1="83.185" x2="64.135" y2="74.93" width="0.8128" layer="16"/>
+<wire x1="64.135" y1="83.5025" x2="64.135" y2="74.93" width="0.8128" layer="16"/>
 <wire x1="64.135" y1="74.93" x2="48.26" y2="74.93" width="0.8128" layer="16"/>
 <wire x1="15.24" y1="13.97" x2="17.78" y2="13.97" width="0.8128" layer="16"/>
@@
 <wire x1="50.8" y1="57.15" x2="52.705" y2="59.055" width="0.8128" layer="16"/>
 <wire x1="52.705" y1="59.055" x2="64.135" y2="59.055" width="0.8128" layer="16"/>
-<wire x1="64.135" y1="83.185" x2="72.39" y2="83.185" width="0.8128" layer="16"/>
-<wire x1="72.39" y1="83.185" x2="73.3425" y2="82.55" width="0.8128" layer="16"/>
-<wire x1="73.3425" y1="82.55" x2="73.3425" y2="64.77" width="0.8128" layer="16"/>
+<wire x1="64.135" y1="83.5025" x2="72.39" y2="83.5025" width="0.8128" layer="16"/>
+<wire x1="72.39" y1="83.5025" x2="73.3425" y2="82.55" width="0.8128" layer="16"/>
+<wire x1="73.3425" y1="82.55" x2="73.3425" y2="74.93" width="0.8128" layer="16"/>
+<wire x1="73.3425" y1="74.93" x2="73.3425" y2="64.77" width="0.8128" layer="16"/>
 <wire x1="48.26" y1="57.15" x2="36.83" y2="57.15" width="0.6096" layer="1"/>
 <wire x1="36.83" y1="57.15" x2="36.83" y2="58.42" width="0.6096" layer="1"/>
 <wire x1="36.83" y1="58.42" x2="34.29" y2="58.42" width="0.6096" layer="1"/>
-<wire x1="64.135" y1="74.93" x2="71.12" y2="74.93" width="0" layer="19" extent="16-16"/>
+<wire x1="71.12" y1="74.93" x2="73.3425" y2="74.93" width="0.8128" layer="16"/>
 </signal>
 <signal name="N$1">
@@
 <wire x1="31.75" y1="39.37" x2="31.75" y2="55.88" width="0.6096" layer="16"/>
 <wire x1="31.75" y1="55.88" x2="34.29" y2="55.88" width="0.6096" layer="16"/>
-<wire x1="48.26" y1="77.47" x2="66.675" y2="77.47" width="0.6096" layer="1"/>
-<wire x1="66.675" y1="77.47" x2="66.675" y2="67.31" width="0.6096" layer="1"/>
-<wire x1="66.675" y1="67.31" x2="71.12" y2="67.31" width="0.6096" layer="1"/>
 <wire x1="53.34" y1="10.16" x2="49.53" y2="13.97" width="0.6096" layer="1"/>
 <wire x1="49.53" y1="13.97" x2="31.75" y2="13.97" width="0.6096" layer="1"/>
@@
 <wire x1="45.72" y1="55.245" x2="45.72" y2="54.61" width="0.6096" layer="1"/>
 <wire x1="45.72" y1="54.61" x2="48.26" y2="54.61" width="0.6096" layer="1"/>
+<wire x1="71.12" y1="67.31" x2="66.675" y2="67.31" width="0.4064" layer="1"/>
+<wire x1="66.675" y1="67.31" x2="66.675" y2="77.47" width="0.4064" layer="1"/>
+<wire x1="66.675" y1="77.47" x2="48.26" y2="77.47" width="0.4064" layer="1"/>
 </signal>
 <signal name="ADC">
@@
 <contactref element="IC1" pad="D4"/>
 <contactref element="LED2" pad="K"/>
-<wire x1="68.58" y1="22.86" x2="68.58" y2="52.07" width="0.6096" layer="16"/>
-<wire x1="68.58" y1="52.07" x2="48.26" y2="52.07" width="0.6096" layer="16"/>
+<wire x1="66.9925" y1="52.07" x2="48.26" y2="52.07" width="0.6096" layer="16"/>
+<wire x1="68.58" y1="22.86" x2="68.58" y2="34.6075" width="0.6096" layer="16"/>
+<wire x1="68.58" y1="34.6075" x2="66.9925" y2="34.6075" width="0.6096" layer="16"/>
+<wire x1="66.9925" y1="34.6075" x2="66.9925" y2="52.07" width="0.6096" layer="16"/>
 </signal>
 <signal name="N$2">
@@
 <wire x1="64.618" y1="22.86" x2="66.04" y2="22.86" width="0.6096" layer="1"/>
 </signal>
+<signal name="N$7">
+<polygon width="0.3048" layer="16" spacing="1.778" isolate="0.8128">
+<vertex x="8.255" y="83.82"/>
+<vertex x="8.255" y="0.3175"/>
+<vertex x="73.66" y="0.3175"/>
+<vertex x="73.66" y="83.82"/>
+</polygon>
+</signal>
+<signal name="N$8">
+<polygon width="0.3048" layer="1" spacing="1.6764" isolate="0.6096">
+<vertex x="8.255" y="83.82"/>
+<vertex x="8.255" y="0.3175"/>
+<vertex x="73.66" y="0.3175"/>
+<vertex x="73.66" y="83.82"/>
+</polygon>
+</signal>
 </signals>
