File: eagle/projekt/projekt.brd (EAGLE design)
At the start: 82 x 84 mm, 20 parts, among them IC1 ESP12E_DEVKIT, IC2 LF50CP, IC3 LEVEL_SHIFTER, IC4 LEVEL_SHIFTER, J1 PSH02-02W

Commit message: Board - podklady
Routing:
- net GND: track 376.6 -> 368.4 mm
- net ADC: track 34.1 -> 33.2 mm
Changed lines of the file:
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@@
 <setting verticaltext="up"/>
 </settings>
-<grid distance="0.0125" unitdist="inch" unit="inch" style="lines" multiple="1" display="no" altdistance="0.025" altunitdist="inch" altunit="inch"/>
+<grid distance="0.0025" unitdist="inch" unit="inch" style="lines" multiple="1" display="no" altdistance="0.025" altunitdist="inch" altunit="inch"/>
 <layers>
 <layer number="1" name="Top" color="4" fill="1" visible="yes" active="yes"/>
@@
 <layer number="17" name="Pads" color="2" fill="1" visible="yes" active="yes"/>
 <layer number="18" name="Vias" color="2" fill="1" visible="yes" active="yes"/>
-<layer number="19" name="Unrouted" color="6" fill="1" visible="no" active="yes"/>
+<layer number="19" name="Unrouted" color="6" fill="1" visible="yes" active="yes"/>
 <layer number="20" name="Dimension" color="15" fill="1" visible="yes" active="yes"/>
 <layer number="21" name="tPlace" color="7" fill="1" visible="yes" active="yes"/>
@@
 <layer number="28" name="bValues" color="7" fill="1" visible="yes" active="yes"/>
 <layer number="29" name="tStop" color="7" fill="3" visible="no" active="yes"/>
-<layer number="30" name="bStop" color="7" fill="6" visible="yes" active="yes"/>
-<layer number="31" name="tCream" color="7" fill="4" visible="yes" active="yes"/>
-<layer number="32" name="bCream" color="7" fill="5" visible="yes" active="yes"/>
-<layer number="33" name="tFinish" color="6" fill="3" visible="yes" active="yes"/>
-<layer number="34" name="bFinish" color="6" fill="6" visible="yes" active="yes"/>
+<layer number="30" name="bStop" color="7" fill="6" visible="no" active="yes"/>
+<layer number="31" name="tCream" color="7" fill="4" visible="no" active="yes"/>
+<layer number="32" name="bCream" color="7" fill="5" visible="no" active="yes"/>
+<layer number="33" name="tFinish" color="6" fill="3" visible="no" active="yes"/>
+<layer number="34" name="bFinish" color="6" fill="6" visible="no" active="yes"/>
 <layer number="35" name="tGlue" color="7" fill="4" visible="no" active="yes"/>
 <layer number="36" name="bGlue" color="7" fill="5" visible="no" active="yes"/>
@@
 <layer number="42" name="bRestrict" color="1" fill="10" visible="no" active="yes"/>
 <layer number="43" name="vRestrict" color="2" fill="10" visible="no" active="yes"/>
-<layer number="44" name="Drills" color="7" fill="1" visible="yes" active="yes"/>
+<layer number="44" name="Drills" color="7" fill="1" visible="no" active="yes"/>
 <layer number="45" name="Holes" color="7" fill="1" visible="yes" active="yes"/>
 <layer number="46" name="Milling" color="3" fill="1" visible="no" active="yes"/>
 <layer number="47" name="Measures" color="7" fill="1" visible="no" active="yes"/>
 <layer number="48" name="Document" color="7" fill="1" visible="yes" active="yes"/>
-<layer number="49" name="Reference" color="7" fill="1" visible="no" active="yes"/>
+<layer number="49" name="Reference" color="7" fill="1" visible="yes" active="yes"/>
 <layer number="50" name="dxf" color="7" fill="1" visible="no" active="no"/>
 <layer number="51" name="tDocu" color="7" fill="1" visible="yes" active="yes"/>
@@
 <wire x1="73.3298" y1="64.77" x2="73.3425" y2="64.77" width="0.6096" layer="16"/>
 <wire x1="73.3298" y1="64.77" x2="71.12" y2="64.77" width="0.8128" layer="16"/>
-<wire x1="64.135" y1="83.5025" x2="64.135" y2="74.93" width="0.8128" layer="16"/>
+<wire x1="64.135" y1="79.121" x2="64.135" y2="74.93" width="0.6096" layer="16"/>
 <wire x1="64.135" y1="74.93" x2="48.26" y2="74.93" width="0.8128" layer="16"/>
 <wire x1="15.24" y1="13.97" x2="17.78" y2="13.97" width="0.8128" layer="16"/>
@@
 <wire x1="50.8" y1="57.15" x2="52.705" y2="59.055" width="0.8128" layer="16"/>
 <wire x1="52.705" y1="59.055" x2="64.135" y2="59.055" width="0.8128" layer="16"/>
-<wire x1="64.135" y1="83.5025" x2="72.39" y2="83.5025" width="0.8128" layer="16"/>
-<wire x1="72.39" y1="83.5025" x2="73.3425" y2="82.55" width="0.8128" layer="16"/>
-<wire x1="73.3425" y1="82.55" x2="73.3425" y2="74.93" width="0.8128" layer="16"/>
-<wire x1="73.3425" y1="74.93" x2="73.3425" y2="64.77" width="0.8128" layer="16"/>
+<wire x1="64.135" y1="79.121" x2="73.3425" y2="79.121" width="0.6096" layer="16"/>
+<wire x1="73.3425" y1="74.93" x2="73.3425" y2="64.77" width="0.6096" layer="16"/>
 <wire x1="48.26" y1="57.15" x2="36.83" y2="57.15" width="0.6096" layer="1"/>
 <wire x1="36.83" y1="57.15" x2="36.83" y2="58.42" width="0.6096" layer="1"/>
 <wire x1="36.83" y1="58.42" x2="34.29" y2="58.42" width="0.6096" layer="1"/>
-<wire x1="71.12" y1="74.93" x2="73.3425" y2="74.93" width="0.8128" layer="16"/>
+<wire x1="71.12" y1="74.93" x2="73.3425" y2="74.93" width="0.6096" layer="16"/>
+<wire x1="73.3425" y1="74.93" x2="73.3425" y2="79.121" width="0.6096" layer="16"/>
 </signal>
 <signal name="N$1">
@@
 <wire x1="33.02" y1="73.66" x2="33.02" y2="77.47" width="0.6096" layer="1"/>
 <wire x1="33.02" y1="77.47" x2="45.72" y2="77.47" width="0.6096" layer="1"/>
-<wire x1="45.72" y1="77.47" x2="45.72" y2="79.375" width="0.6096" layer="1"/>
-<wire x1="45.72" y1="79.375" x2="60.96" y2="79.375" width="0.6096" layer="1"/>
+<wire x1="45.72" y1="77.47" x2="46.99" y2="79.0575" width="0.6096" layer="1"/>
 <wire x1="60.96" y1="79.375" x2="60.96" y2="78.892" width="0.4064" layer="1"/>
+<wire x1="46.99" y1="78.994" x2="46.99" y2="79.0575" width="0.6096" layer="1"/>
+<wire x1="46.99" y1="79.0575" x2="60.96" y2="79.0575" width="0.6096" layer="1"/>
+<wire x1="60.96" y1="79.0575" x2="60.96" y2="78.892" width="0.4064" layer="1"/>
 </signal>
 <signal name="RST">
