File: eagle/projekt/mod_temperature.sch (EAGLE design)
At the start: 2 parts

Commit message: Cidlo teploty
Parts:
- added C1: 100n, rcl:C-EU025-025X050
- added JP1: (no value), SparkFun-Connectors:M08X2
- added R1: 4k7, rcl:R-EU_0207/10
- U1: value (none) -> DHT22
Connections:
- new net GND: C1.2, PL1.14, U1.GND
- new net GPIO1: JP1.1, PL1.3
- new net GPIO12: JP1.9, PL1.7
- new net GPIO13: JP1.11, PL1.8
- new net GPIO14: JP1.13, PL1.9
- new net GPIO16: JP1.15, PL1.10
- new net GPIO3: JP1.3, PL1.4
- new net GPIO4: JP1.5, PL1.5
- new net GPIO5: JP1.7, PL1.6
- new net N$2: JP1.10, JP1.12, JP1.14, JP1.16, JP1.2, JP1.4, JP1.6, JP1.8, R1.1, U1.DATA
- new net VCC: C1.1, PL1.1, R1.2, U1.VDD
Other:
- moved on the sheet: PL1, U1
