File: eagle/projekt/mod_io.sch (EAGLE design)
At the start: 20 parts, among them IC1 PCF8574T

Commit message: Update schematu
Parts:
- removed JP1, JP2, JP3, JP4: (no value), SparkFun-Connectors:M08X2
- removed JP5: (no value), SparkFun-Connectors:M03LONGPADS
- removed JP8: (no value), SparkFun-Connectors:M08
- removed PL2: (no value), con-harting-v:14V
- removed X1: (no value), con-ptr500+:AK550/8
- added A3: (no value), SparkFun-Connectors:M03LONGPADS
- added CNF4, INT, SCL, SDA: (no value), SparkFun-Connectors:M08LONGPADS
- added D1, D2, D3, D4, D5, D6, D7, D8: L-53LSRD, SparkFun-LED:LED5MM
- added IO2: (no value), con-harting-v:14V
- added IO3: (no value), SparkFun-Connectors:M10LOCK_LONGPADS
- added IO4: (no value), con-ptr500+:AK550/10
- added R1, R2, R3, R4, R7, R8: 1k6, resistor:R-EU_0207/10
- added R10, R11, R12, R13, R14, R15, R16, R9: 10k, resistor:R-EU_0207/10
- added R17, R18: 4k7, resistor:R-EU_0207/10
- added R5, R6: (no value), resistor:R-EU_0207/10
- renumbered JP6 to A1, JP7 to A2, PL1 to IO1
Connections:
- new net GND: IC1.VSS, S1.P, S1.P@1, S2.P, S2.P@1, S3.P, S3.P@1, S4.P, S4.P@1, S5.P, S5.P@1, S6.P, S6.P@1, S7.P, S7.P@1, S8.P, S8.P@1
- new net N$17: IC1.!INT, INT.1, INT.2, INT.3, INT.4, INT.5, INT.6, INT.7, INT.8
- new net N$18: A3.3, IC1.A0
- new net N$19: A3.2, IC1.A1
- new net N$20: A3.1, IC1.A2
- new net N$21: IC1.SDA, R17.2
- new net N$22: IC1.SCL, R18.2
- new net N$23: R17.1, SDA.1, SDA.2, SDA.3, SDA.4, SDA.5, SDA.6, SDA.7, SDA.8
- new net N$25: R18.1, SCL.1, SCL.2, SCL.3, SCL.4, SCL.5, SCL.6, SCL.7, SCL.8
- new net VCC: IC1.VDD, R1.2, R10.2, R11.2, R12.2, R13.2, R14.2, R15.2, R16.2, R2.2, R3.2, R4.2, R5.2, R6.2, R7.2, R8.2, R9.2
- net N$1: now also D5.C, IC1.P4, R13.1, S5.S, S5.S@1; no longer JP3.1, JP4.1
- net N$10: now also D5.A, R5.1; no longer JP3.10, JP4.10
- net N$11: now also D7.A, R7.1; no longer JP3.11, JP4.11
- net N$12: now also D8.A, R8.1; no longer JP3.12, JP4.12
- net N$13: now also D1.A, R1.1; no longer JP3.13, JP4.13
- net N$14: now also D2.A, R2.1; no longer JP3.14, JP4.14
- net N$15: now also D3.A, R3.1; no longer JP3.15, JP4.15
- net N$16: now also D4.A, R4.1; no longer JP3.16, JP4.16
- net N$2: now also D6.C, IC1.P5, R14.1, S6.S, S6.S@1; no longer JP3.2, JP4.2
- net N$3: now also D1.C, IC1.P0, R9.1, S1.S, S1.S@1; no longer JP3.3, JP4.3
- net N$4: now also D2.C, IC1.P1, R10.1, S2.S, S2.S@1; no longer JP3.4, JP4.4
- net N$5: now also D3.C, IC1.P2, R11.1, S3.S, S3.S@1; no longer JP3.5, JP4.5
- net N$6: now also D4.C, IC1.P3, R12.1, S4.S, S4.S@1; no longer JP3.6, JP4.6
- net N$7: now also D7.C, IC1.P6, R15.1, S7.S, S7.S@1; no longer JP3.7, JP4.7
- net N$8: now also D8.C, IC1.P7, R16.1, S8.S, S8.S@1; no longer JP3.8, JP4.8
- net N$9: now also D6.A, R6.1; no longer JP3.9, JP4.9
Other:
- moved on the sheet: IC1, S1, S2, S3, S4, S5, S6, S7, S8

Commit message: Update schematu
Parts:
- added C1: 100n, rcl:C-EU050-025X075
Connections:
- new net 3V3: IO1.2, IO2.2
- new net ADC: IO1.12, IO2.12
- new net GPIO1: CNF4.1, IO1.3, IO2.3
- new net GPIO12: CNF4.5, IO1.7, IO2.7
- new net GPIO13: CNF4.6, IO1.8, IO2.8
- new net GPIO14: CNF4.7, IO1.9, IO2.9
- new net GPIO16: CNF4.8, IO1.10, IO2.10
- new net GPIO3: CNF4.2, IO1.4, IO2.4
- new net GPIO4: CNF4.3, IO1.5, IO2.5
- new net GPIO5: CNF4.4, IO1.6, IO2.6
- new net RST: IO1.11, IO2.11
- new net VIN: IO1.13, IO2.13
- net GND: now also A2.1, A2.2, A2.3, C1.2, IO1.14, IO2.14, IO3.10, IO4-10.KL
- net N$1: now also IO3.6, IO4-6.KL
- net N$2: now also IO3.7, IO4-7.KL
- net N$3: now also IO3.2, IO4-2.KL
- net N$4: now also IO3.3, IO4-3.KL
- net N$5: now also IO3.4, IO4-4.KL
- net N$6: now also IO3.5, IO4-5.KL
- net N$7: now also IO3.8, IO4-8.KL
- net N$8: now also IO3.9, IO4-9.KL
- net VCC: now also A1.1, A1.2, A1.3, C1.1, IO1.1, IO2.1, IO3.1, IO4-1.KL
Other:
- moved on the sheet: A1, A2, A3, CNF4, D1, D2, D3, D4, D5, D6, D7, D8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

Commit message: Update schematu
Parts:
- IC1: value PCF8574T -> PCF8574P; device micro-philips:PCF8574T -> micro-philips:PCF8574P
- IO3: value (none) -> PINHD-1X10; device SparkFun-Connectors:M10LOCK_LONGPADS -> adafruit:PINHD-1X10
- renumbered CNF4 to CNF
Other:
- moved on the sheet: IO3
